File: mcu-proto-100x68mm/MCU_PROTO_100x68mm.kicad_sch (KiCad schematic)
At the start: 4 parts, among them J1 Screw_Terminal_01x04, J2 Screw_Terminal_01x04, J3 Conn_01x01_Pin, J4 Conn_01x01_Pin

Commit message: Silkscreen on front side
Connections:
- net GND: now reaches J3.1 (Pin_1), J4.1 (Pin_1)
Changed lines of the file:
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@@
     (company "Galopago")
   )
+  (junction (at 196.85 40.64) (diameter 0) (color 0 0 0 0)
+  )
   (wire (pts (xy 190.5 40.64) (xy 196.85 40.64))
+    (stroke (width 0) (type default))
+  )
+  (wire (pts (xy 200.66 40.64) (xy 200.66 41.91))
+    (stroke (width 0) (type default))
+  )
+  (wire (pts (xy 196.85 40.64) (xy 200.66 40.64))
     (stroke (width 0) (type default))
   )
@@
         )
       )
+    )
+  )
+  (symbol (lib_id "power:GND") (at 200.66 41.91 0) (unit 1)
+    (in_bom yes) (on_board yes) (dnp no) (fields_autoplaced)
+    (property "Reference" "#PWR01" (at 200.66 48.26 0)
+      (effects (font (size 1.27 1.27)) hide)
+    )
+    (property "Value" "GND" (at 200.66 46.99 0)
+      (effects (font (size 1.27 1.27)))
+    )
+    (property "Footprint" "" (at 200.66 41.91 0)
+      (effects (font (size 1.27 1.27)) hide)
+    )
+    (property "Datasheet" "" (at 200.66 41.91 0)
+      (effects (font (size 1.27 1.27)) hide)
+    )
+    (pin "1")
+    (instances
+      (project "MCU_PROTO_100x68mm"
+        (path "/76e65cbe-b273-4a09-a4a4-1a589f3b5a37"
+          (reference "#PWR01") (unit 1)
+        )
+      )
